File: v01/eagle/lighthouse-v01/lighthouse-v01.sch (EAGLE design)
At the start: 65 parts, among them IC1 FT232RLSSOP, U1 TLC5940PWP, U2 TLC5940PWP, U3 TLC5940PWP, U4 SN74LVC244A-TSSOP, U5 ATMEGA644A-AU, U6 WIZ820IO, U7 AOZ1280CI, U8 SN74LVC1G125-SOT23-5, X1 USBSMD

Commit message: Changed TSSOP-28 Reference
Parts:
- U1, U2, U3: EAGLEUP TSSOP-28-POWERPAD -> TSSOP-28
Changed lines of the file:
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@@
 <parts>
 <part name="U1" library="SparkFun" deviceset="TLC5940" device="PWP">
-<attribute name="EAGLEUP" value="TSSOP-28-POWERPAD"/>
+<attribute name="EAGLEUP" value="TSSOP-28"/>
 </part>
 <part name="GND1" library="SparkFun" deviceset="GND" device=""/>
@@
 <part name="GND25" library="SparkFun" deviceset="GND" device=""/>
 <part name="U2" library="SparkFun" deviceset="TLC5940" device="PWP">
-<attribute name="EAGLEUP" value="TSSOP-28-POWERPAD"/>
+<attribute name="EAGLEUP" value="TSSOP-28"/>
 </part>
 <part name="GND2" library="SparkFun" deviceset="GND" device=""/>
@@
 <part name="GND3" library="SparkFun" deviceset="GND" device=""/>
 <part name="U3" library="SparkFun" deviceset="TLC5940" device="PWP">
-<attribute name="EAGLEUP" value="TSSOP-28-POWERPAD"/>
+<attribute name="EAGLEUP" value="TSSOP-28"/>
 </part>
 <part name="GND12" library="SparkFun" deviceset="GND" device=""/>
